Commit message: finalproject

File: body.urdf (robot description, URDF)
Before this commit: robot robot, 9 links, 8 joints
Links:
- removed link BackLeg
- removed link BackLowerLeg
- removed link FrontLeg
- removed link FrontLowerLeg
- removed link LeftLeg
- removed link LeftLowerLeg
- removed link RightLeg
- removed link RightLowerLeg
- added link BackLeftFoot, mass 1; collision box size=0.2 0.2 0.5; visual box size=0.2 0.2 0.5
- added link BackLeftLeg, mass 1; collision box size=0.2 0.5 0.2; visual box size=0.2 0.5 0.2
- added link BackRightFoot, mass 1; collision box size=0.2 0.2 0.5; visual box size=0.2 0.2 0.5
- added link BackRightLeg, mass 1; collision box size=0.2 0.5 0.2; visual box size=0.2 0.5 0.2
- added link FrontLeftFoot, mass 1; collision box size=0.2 0.2 0.5; visual box size=0.2 0.2 0.5
- added link FrontLeftLeg, mass 1; collision box size=0.2 0.5 0.2; visual box size=0.2 0.5 0.2
- added link FrontRightFoot, mass 1; collision box size=0.2 0.2 0.5; visual box size=0.2 0.2 0.5
- added link FrontRightLeg, mass 1; collision box size=0.2 0.5 0.2; visual box size=0.2 0.5 0.2
- added link MiddleLeftFoot, mass 1; collision box size=0.2 0.2 0.5; visual box size=0.2 0.2 0.5
- added link MiddleLeftLeg, mass 1; collision box size=0.2 0.5 0.2; visual box size=0.2 0.5 0.2
- added link MiddleRightFoot, mass 1; collision box size=0.2 0.2 0.5; visual box size=0.2 0.2 0.5
- added link MiddleRightLeg, mass 1; collision box size=0.2 0.5 0.2; visual box size=0.2 0.5 0.2
- link Torso: geometry collision box size=2 0.5 0.5; visual box size=2 0.5 0.5
Joints:
- removed joint BackLeg_BackLowerLeg
- removed joint FrontLeg_FrontLowerLeg
- removed joint LeftLeg_LeftLowerLeg
- removed joint RightLeg_RightLowerLeg
- removed joint Torso_BackLeg
- removed joint Torso_FrontLeg
- removed joint Torso_LeftLeg
- removed joint Torso_RightLeg
- added joint BackLeftLeg_BackLeftFoot: type revolute, parent BackLeftLeg, child BackLeftFoot, origin xyz=0 -0.5 0 rpy=0 0 0, axis 1 0 0, limit lower=-3.14159 upper=3.14159 effort=0.0 velocity=0.0
- added joint BackRightLeg_BackRightFoot: type revolute, parent BackRightLeg, child BackRightFoot, origin xyz=0 0.5 0 rpy=0 0 0, axis 1 0 0, limit lower=-3.14159 upper=3.14159 effort=0.0 velocity=0.0
- added joint FrontLeftLeg_FrontLeftFoot: type revolute, parent FrontLeftLeg, child FrontLeftFoot, origin xyz=0 -0.5 0 rpy=0 0 0, axis 1 0 0, limit lower=-3.14159 upper=3.14159 effort=0.0 velocity=0.0
- added joint FrontRightLeg_FrontRightFoot: type revolute, parent FrontRightLeg, child FrontRightFoot, origin xyz=0 0.5 0 rpy=0 0 0, axis 1 0 0, limit lower=-3.14159 upper=3.14159 effort=0.0 velocity=0.0
- added joint MiddleLeftLeg_MiddleLeftFoot: type revolute, parent MiddleLeftLeg, child MiddleLeftFoot, origin xyz=0 -0.5 0 rpy=0 0 0, axis 1 0 0, limit lower=-3.14159 upper=3.14159 effort=0.0 velocity=0.0
- added joint MiddleRightLeg_MiddleRightFoot: type revolute, parent MiddleRightLeg, child MiddleRightFoot, origin xyz=0 0.5 0 rpy=0 0 0, axis 1 0 0, limit lower=-3.14159 upper=3.14159 effort=0.0 velocity=0.0
- added joint Torso_BackLeftLeg: type revolute, parent Torso, child BackLeftLeg, origin xyz=0.5 -0.25 0.5 rpy=0 0 0, axis 1 0 0, limit lower=-3.14159 upper=3.14159 effort=0.0 velocity=0.0
- added joint Torso_BackRightLeg: type revolute, parent Torso, child BackRightLeg, origin xyz=0.5 0.25 0.5 rpy=0 0 0, axis 1 0 0, limit lower=-3.14159 upper=3.14159 effort=0.0 velocity=0.0
- added joint Torso_FrontLeftLeg: type revolute, parent Torso, child FrontLeftLeg, origin xyz=-0.5 -0.25 0.5 rpy=0 0 0, axis 1 0 0, limit lower=-3.14159 upper=3.14159 effort=0.0 velocity=0.0
- added joint Torso_FrontRightLeg: type revolute, parent Torso, child FrontRightLeg, origin xyz=-0.5 0.25 0.5 rpy=0 0 0, axis 1 0 0, limit lower=-3.14159 upper=3.14159 effort=0.0 velocity=0.0
- added joint Torso_MiddleLeftLeg: type revolute, parent Torso, child MiddleLeftLeg, origin xyz=0 -0.25 0.5 rpy=0 0 0, axis 1 0 0, limit lower=-3.14159 upper=3.14159 effort=0.0 velocity=0.0
- added joint Torso_MiddleRightLeg: type revolute, parent Torso, child MiddleRightLeg, origin xyz=0 0.25 0.5 rpy=0 0 0, axis 1 0 0, limit lower=-3.14159 upper=3.14159 effort=0.0 velocity=0.0

Commit message: done

File: body.urdf (robot description, URDF)
Before this commit: robot robot, 13 links, 12 joints
Links:
- removed link BackLeftFoot
- removed link BackLeftLeg
- removed link BackRightFoot
- removed link BackRightLeg
- removed link FrontLeftFoot
- removed link FrontLeftLeg
- removed link FrontRightFoot
- removed link FrontRightLeg
- removed link MiddleLeftFoot
- removed link MiddleLeftLeg
- removed link MiddleRightFoot
- removed link MiddleRightLeg
- removed link Torso
- added link 0, mass 1; collision box size=0.4335664189053008 0.6247815058846707 0.7149500523886889; visual box size=0.4335664189053008 0.6247815058846707 0.7149500523886889
- added link 1, mass 1; collision box size=1.3379871247856088 0.8173365057416286 0.9758742320429974; visual box size=1.3379871247856088 0.8173365057416286 0.9758742320429974
- added link 2, mass 1; collision box size=1.4812859428090248 0.8550219911965142 0.9034085257827643; visual box size=1.4812859428090248 0.8550219911965142 0.9034085257827643
- added link 3, mass 1; collision box size=0.3606098033834566 0.5216485508745126 0.6342865081033173; visual box size=0.3606098033834566 0.5216485508745126 0.6342865081033173
- added link 4, mass 1; collision box size=1.1569456980384227 0.7739011150224313 0.5286106396861474; visual box size=1.1569456980384227 0.7739011150224313 0.5286106396861474
- added link 5, mass 1; collision box size=0.7421018986659726 0.904797559420718 0.6655129261773949; visual box size=0.7421018986659726 0.904797559420718 0.6655129261773949
Joints:
- removed joint BackLeftLeg_BackLeftFoot
- removed joint BackRightLeg_BackRightFoot
- removed joint FrontLeftLeg_FrontLeftFoot
- removed joint FrontRightLeg_FrontRightFoot
- removed joint MiddleLeftLeg_MiddleLeftFoot
- removed joint MiddleRightLeg_MiddleRightFoot
- removed joint Torso_BackLeftLeg
- removed joint Torso_BackRightLeg
- removed joint Torso_FrontLeftLeg
- removed joint Torso_FrontRightLeg
- removed joint Torso_MiddleLeftLeg
- removed joint Torso_MiddleRightLeg
- added joint 0_1: type revolute, parent 0, child 1, origin xyz=-0.2167832094526504 0 0.5 rpy=0 0 0, axis 0 0 1, limit lower=-3.14159 upper=3.14159 effort=0.0 velocity=0.0
- added joint 1_2: type revolute, parent 1, child 2, origin xyz=-1.3379871247856088 0 0 rpy=0 0 0, axis 0 0 1, limit lower=-3.14159 upper=3.14159 effort=0.0 velocity=0.0
- added joint 2_3: type revolute, parent 2, child 3, origin xyz=-1.4812859428090248 0 0 rpy=0 0 0, axis 0 0 1, limit lower=-3.14159 upper=3.14159 effort=0.0 velocity=0.0
- added joint 3_4: type revolute, parent 3, child 4, origin xyz=-0.3606098033834566 0 0 rpy=0 0 0, axis 0 0 1, limit lower=-3.14159 upper=3.14159 effort=0.0 velocity=0.0
- added joint 4_5: type revolute, parent 4, child 5, origin xyz=-1.1569456980384227 0 0 rpy=0 0 0, axis 0 0 1, limit lower=-3.14159 upper=3.14159 effort=0.0 velocity=0.0

Commit message: random 3D

File: body.urdf (robot description, URDF)
Before this commit: robot robot, 6 links, 5 joints
Links:
- added link 6, mass 1; collision box size=0.5970102714633713 0.15491658078745485 0.9047070611991346; visual box size=0.5970102714633713 0.15491658078745485 0.9047070611991346
- added link 7, mass 1; collision box size=0.3638512395419774 0.9799145366009333 0.7276441650436503; visual box size=0.3638512395419774 0.9799145366009333 0.7276441650436503
- link 0: geometry collision box size=0.18643094120200387 0.5062827968575684 0.9190824504345745; visual box size=0.18643094120200387 0.5062827968575684 0.9190824504345745
- link 1: geometry collision box size=0.0017420619330478226 0.8738946058838928 0.8359164747140165; visual box size=0.0017420619330478226 0.8738946058838928 0.8359164747140165
- link 2: geometry collision box size=0.045350575310111996 0.7050758702936072 0.6000969532912857; visual box size=0.045350575310111996 0.7050758702936072 0.6000969532912857
- link 3: geometry collision box size=0.6348345818008763 0.12834038184565955 0.45760935258611746; visual box size=0.6348345818008763 0.12834038184565955 0.45760935258611746
- link 4: geometry collision box size=0.8687506572754338 0.5119926290823207 0.8358103235733981; visual box size=0.8687506572754338 0.5119926290823207 0.8358103235733981
- link 5: geometry collision box size=0.4834981234375755 0.5824795856147429 0.5142774646056034; visual box size=0.4834981234375755 0.5824795856147429 0.5142774646056034
Joints:
- removed joint 1_2
- removed joint 2_3
- removed joint 3_4
- removed joint 4_5
- added joint 0_2: type revolute, parent 0, child 2, origin xyz=0 0 0.4138941609710629 rpy=0 0 0, axis 1 0 0, limit lower=-3.14159 upper=3.14159 effort=0.0 velocity=0.0
- added joint 0_3: type revolute, parent 0, child 3, origin xyz=-0.09321547060100194 0 0.8734353861883501 rpy=0 0 0, axis 0 0 1, limit lower=-3.14159 upper=3.14159 effort=0.0 velocity=0.0
- added joint 0_4: type revolute, parent 0, child 4, origin xyz=0 0 1.3329766114056374 rpy=0 0 0, axis 0 0 1, limit lower=-3.14159 upper=3.14159 effort=0.0 velocity=0.0
- added joint 3_5: type revolute, parent 3, child 5, origin xyz=-0.31741729090043813 0 0.22880467629305867 rpy=0 0 0, axis 1 0 0, limit lower=-3.14159 upper=3.14159 effort=0.0 velocity=0.0
- added joint 5_6: type revolute, parent 5, child 6, origin xyz=0.0 0.29123979280737144 0.2571387323028016 rpy=0 0 0, axis 1 0 0, limit lower=-3.14159 upper=3.14159 effort=0.0 velocity=0.0
- added joint 6_7: type revolute, parent 6, child 7, origin xyz=-0.29850513573168563 0.07745829039372742 0.0 rpy=0 0 0, axis 0 1 0, limit lower=-3.14159 upper=3.14159 effort=0.0 velocity=0.0
- joint 0_1: origin xyz=-0.2167832094526504 0 0.5 rpy=0 0 0 -> xyz=0 -0.2531413984287842 0.8734353861883501 rpy=0 0 0

Commit message: updates

File: body.urdf (robot description, URDF)
Before this commit: robot robot, 8 links, 7 joints
Links:
- removed link 6
- removed link 7
- link 0: geometry collision box size=0.7660321367165701 0.3865805453424317 0.19186975109939708; visual box size=0.7660321367165701 0.3865805453424317 0.19186975109939708
- link 1: geometry collision box size=0.208373533474688 0.3243337895712066 0.4756428656593893; visual box size=0.208373533474688 0.3243337895712066 0.4756428656593893
- link 2: geometry collision box size=0.034454087043299 0.3633758205799028 0.9095921452472359; visual box size=0.034454087043299 0.3633758205799028 0.9095921452472359
- link 3: geometry collision box size=0.23359896398518476 0.9819441893386724 0.32957580100889605; visual box size=0.23359896398518476 0.9819441893386724 0.32957580100889605
- link 4: geometry collision box size=0.38679171762457354 0.23550292066631762 0.7247384634714087; visual box size=0.38679171762457354 0.23550292066631762 0.7247384634714087
- link 5: geometry collision box size=0.8649323862201383 0.28865697657698575 0.4306603490876868; visual box size=0.8649323862201383 0.28865697657698575 0.4306603490876868
Joints:
- removed joint 0_2
- removed joint 0_3
- removed joint 0_4
- removed joint 5_6
- removed joint 6_7
- added joint 1_2: type revolute, parent 1, child 2, origin xyz=0.208373533474688 0 0.0 rpy=0 0 0, axis 1 0 0, limit lower=-3.14159 upper=3.14159 effort=0.0 velocity=0.0
- added joint 1_3: type revolute, parent 1, child 3, origin xyz=0.104186766737344 -0.1621668947856033 0.0 rpy=0 0 0, axis 0 1 0, limit lower=-3.14159 upper=3.14159 effort=0.0 velocity=0.0
- added joint 2_4: type revolute, parent 2, child 4, origin xyz=0.0172270435216495 -0.1816879102899514 0.0 rpy=0 0 0, axis 0 1 0, limit lower=-3.14159 upper=3.14159 effort=0.0 velocity=0.0
- joint 0_1: axis 0 0 1 -> 1 0 0; origin xyz=0 -0.2531413984287842 0.8734353861883501 rpy=0 0 0 -> xyz=0.38301606835828506 0 0.9564708164550441 rpy=0 0 0
- joint 3_5: axis 1 0 0 -> 0 1 0; origin xyz=-0.31741729090043813 0 0.22880467629305867 rpy=0 0 0 -> xyz=-0.11679948199259238 -0.4909720946693362 0.0 rpy=0 0 0
