Commit message: done

File: saved_configs/body0.urdf (robot description, URDF)
Before this commit: robot robot, 6 links, 5 joints
Links:
- link 0: geometry collision box size=0.4789704272179115 0.4754548494172842 0.4616790242162536; visual box size=0.4789704272179115 0.4754548494172842 0.4616790242162536
- link 1: geometry collision box size=0.14093231374026227 0.35670821153115884 0.11543126812360216; visual box size=0.14093231374026227 0.35670821153115884 0.11543126812360216
- link 2: geometry collision box size=0.4085433370842445 0.4080109801314763 0.551457015979915; visual box size=0.4085433370842445 0.4080109801314763 0.551457015979915
- link 3: geometry collision box size=0.4788213833321736 0.8595400955799134 0.8767560111669435; visual box size=0.4788213833321736 0.8595400955799134 0.8767560111669435
- link 4: geometry collision box size=0.91849245140848 0.27918011073456594 0.968489589975287; visual box size=0.91849245140848 0.27918011073456594 0.968489589975287
- link 5: geometry collision box size=0.018863019451183294 0.5867544693601409 0.9526315745990082; visual box size=0.018863019451183294 0.5867544693601409 0.9526315745990082
Joints:
- removed joint 1_2
- removed joint 2_4
- removed joint 3_5
- added joint 0_2: type revolute, parent 0, child 2, origin xyz=-0.23948521360895575 0 1.203353507479663 rpy=0 0 0, axis 1 0 0, limit lower=-3.14159 upper=3.14159 effort=0.0 velocity=0.0
- added joint 1_4: type revolute, parent 1, child 4, origin xyz=0.07046615687013114 0 -0.057715634061801024 rpy=0 0 0, axis 1 0 0, limit lower=-3.14159 upper=3.14159 effort=0.0 velocity=0.0
- added joint 1_5: type revolute, parent 1, child 5, origin xyz=0.07046615687013114 -0.17835410576557942 0.0 rpy=0 0 0, axis 0 1 0, limit lower=-3.14159 upper=3.14159 effort=0.0 velocity=0.0
- joint 0_1: axis 1 0 0 -> 0 1 0; origin xyz=0.38301606835828506 0 0.9564708164550441 rpy=0 0 0 -> xyz=0.23948521360895575 0 1.203353507479663 rpy=0 0 0
- joint 1_3: origin xyz=0.104186766737344 -0.1621668947856033 0.0 rpy=0 0 0 -> xyz=0.14093231374026227 0 0.0 rpy=0 0 0
